Commit message: Moveit package for 3F UR5e with new URDF model

File: catkin_ws/src/ur5eRobotiq3f_moveit_config/config/gazebo_ur5e_robot.urdf (robot description, URDF)
Before this commit: robot ur5e_robot, 39 links, 38 joints
Links:
- added link base_link_inertia, mass 4.0; collision mesh filename=package://ur_description/meshes/ur5e/collision/base.stl; visual mesh filename=package://ur_description/meshes/ur5e/visual/base.dae
- added link flange
- link base_link: mass 4.0 -> None; geometry 
- link ee_link: mass 0.1 -> None; geometry 
- link forearm_link: geometry collision mesh filename=package://ur_description/meshes/ur5e/collision/forearm.stl; visual mesh filename=package://ur_description/meshes/ur5e/visual/forearm.dae
- link shoulder_link: geometry collision mesh filename=package://ur_description/meshes/ur5e/collision/shoulder.stl; visual mesh filename=package://ur_description/meshes/ur5e/visual/shoulder.dae
- link table: mass 1000 -> 50
- link upper_arm_link: geometry collision mesh filename=package://ur_description/meshes/ur5e/collision/upperarm.stl; visual mesh filename=package://ur_description/meshes/ur5e/visual/upperarm.dae
- link wrist_1_link: geometry collision mesh filename=package://ur_description/meshes/ur5e/collision/wrist1.stl; visual mesh filename=package://ur_description/meshes/ur5e/visual/wrist1.dae
- link wrist_2_link: geometry collision mesh filename=package://ur_description/meshes/ur5e/collision/wrist2.stl; visual mesh filename=package://ur_description/meshes/ur5e/visual/wrist2.dae
- link wrist_3_link: geometry collision mesh filename=package://ur_description/meshes/ur5e/collision/wrist3.stl; visual mesh filename=package://ur_description/meshes/ur5e/visual/wrist3.dae
Joints:
- removed joint ee_fixed_joint
- removed joint wrist_3_link-tool0_fixed_joint
- added joint base_link-base_link_inertia: type fixed, parent base_link, child base_link_inertia, origin xyz=0 0 0 rpy=0 0 3.141592653589793
- added joint flange-tool0: type fixed, parent flange, child tool0, origin xyz=0 0 0 rpy=1.5707963267948966 0 1.5707963267948966
- added joint tool0_ee_link: type fixed, parent tool0, child ee_link, origin xyz=0 0 0 rpy=0 0 0
- added joint wrist_3-flange: type fixed, parent wrist_3_link, child flange, origin xyz=0 0 0 rpy=0 -1.5707963267948966 -1.5707963267948966
- joint base_link-base_fixed_joint: origin xyz=0 0 0 rpy=0 0 -3.141592653589793 -> xyz=0 0 0 rpy=0 0 3.141592653589793
- joint base_robot_joint: origin xyz=0.0 0.0 0.35 rpy=0.0 0.0 0.0 -> xyz=0.0 0.0 0.35 rpy=0.0 0.0 -1.57
- joint camera_joint: origin xyz=0.05472 0.014 0.03 rpy=3.1414 0.0 1.5707 -> xyz=0.055 0.015 0.03 rpy=3.1414 0.0 1.5707
- joint elbow_joint: axis 0 1 0 -> 0 0 1; limit lower=-3.141592653589793 upper=3.141592653589793 effort=150.0 velocity=3.14 -> lower=-3.141592653589793 upper=3.141592653589793 effort=150.0 velocity=3.141592653589793; origin xyz=0.0 -0.131 0.425 rpy=0.0 0.0 0.0 -> xyz=-0.425 0 0 rpy=0 0 0
- joint shoulder_lift_joint: axis 0 1 0 -> 0 0 1; limit lower=-3.141592653589793 upper=3.141592653589793 effort=150.0 velocity=3.14 -> lower=-6.283185307179586 upper=6.283185307179586 effort=150.0 velocity=3.141592653589793; origin xyz=0.0 0.138 0.0 rpy=0.0 1.5707963267948966 0.0 -> xyz=0 0 0 rpy=1.570796327 0 0
- joint shoulder_pan_joint: limit lower=-3.141592653589793 upper=3.141592653589793 effort=150.0 velocity=3.14 -> lower=-6.283185307179586 upper=6.283185307179586 effort=150.0 velocity=3.141592653589793; origin xyz=0.0 0.0 0.163 rpy=0.0 0.0 0.0 -> xyz=0 0 0.1625 rpy=0 0 0; parent base_link -> base_link_inertia
- joint urGripper_gripper_joint: origin xyz=0.05355 0.05 0.17247 rpy=0.0 3.1415 0.0 -> xyz=0.055 0.068 0.1735 rpy=0.0 3.14 0.0
- joint ur_gripper_joint: origin xyz=-0.002 -0.08423 -0.15968 rpy=0.0 -0.7854 -1.57 -> xyz=0.08423 0.161 -0.0 rpy=1.57 -0.0 -0.785; parent ee_link -> wrist_3_link
- joint wrist_1_joint: axis 0 1 0 -> 0 0 1; limit lower=-3.141592653589793 upper=3.141592653589793 effort=28.0 velocity=6.28 -> lower=-6.283185307179586 upper=6.283185307179586 effort=28.0 velocity=3.141592653589793; origin xyz=0.0 0.0 0.392 rpy=0.0 1.5707963267948966 0.0 -> xyz=-0.3922 0 0.1333 rpy=0 0 0
- joint wrist_2_joint: limit lower=-3.141592653589793 upper=3.141592653589793 effort=28.0 velocity=6.28 -> lower=-6.283185307179586 upper=6.283185307179586 effort=28.0 velocity=3.141592653589793; origin xyz=0.0 0.127 0.0 rpy=0.0 0.0 0.0 -> xyz=0 -0.0997 -2.044881182297852e-11 rpy=1.570796327 0 0
- joint wrist_3_joint: axis 0 1 0 -> 0 0 1; limit lower=-3.141592653589793 upper=3.141592653589793 effort=28.0 velocity=6.28 -> lower=-6.283185307179586 upper=6.283185307179586 effort=28.0 velocity=3.141592653589793; origin xyz=0.0 0.0 0.1 rpy=0.0 0.0 0.0 -> xyz=0 0.0996 -2.042830148012698e-11 rpy=1.570796326589793 3.141592653589793 3.141592653589793
