Commit message: Using original UR5e URDF model
Use the URDF model that is loaded with Moveit!

File: catkin_ws/src/experiment_settings/urdf/ur5e_sim.xacro (robot description, xacro)
@@ -4,5 +4,5 @@
 <!-- |    EDITING THIS FILE BY HAND IS NOT RECOMMENDED                                 | -->
 <!-- =================================================================================== -->
-<robot name="ur5e_robot">
+<robot name="ur5e_robot" xmlns:xacro="http://wiki.ros.org/xacro">
   <gazebo>
     <plugin filename="libgazebo_ros_control.so" name="gazebo_ros_control">
@@ -40,270 +40,22 @@
   <!--property name="wrist_3_length" value="0.0823" /-->
   <!-- manually measured -->
-  <link name="base_link">
-    <visual>
-      <geometry>
-        <mesh filename="package://experiment_settings/meshes/visual/base.dae"/>
-      </geometry>
-      <material name="LightGrey">
-        <color rgba="0.7 0.7 0.7 1.0"/>
-      </material>
-    </visual>
-    <collision>
-      <geometry>
-        <mesh filename="package://experiment_settings/meshes/collision/base.stl"/>
-      </geometry>
-    </collision>
-    <inertial>
-      <mass value="4.0"/>
-      <origin rpy="0 0 0" xyz="0.0 0.0 0.0"/>
-      <inertia ixx="0.00443333156" ixy="0.0" ixz="0.0" iyy="0.00443333156" iyz="0.0" izz="0.0072"/>
-    </inertial>
-  </link>
-  <joint name="shoulder_pan_joint" type="revolute">
-    <parent link="base_link"/>
-    <child link="shoulder_link"/>
-    <origin rpy="0.0 0.0 0.0" xyz="0.0 0.0 0.163"/>
-    <axis xyz="0 0 1"/>
-    <limit effort="150.0" lower="-3.141592653589793" upper="3.141592653589793" velocity="3.14"/>
-    <dynamics damping="0.0" friction="0.0"/>
-  </joint>
-  <link name="shoulder_link">
-    <visual>
-      <geometry>
-        <mesh filename="package://experiment_settings/meshes/visual/shoulder.dae"/>
-      </geometry>
-      <material name="LightGrey">
-        <color rgba="0.7 0.7 0.7 1.0"/>
-      </material>
-    </visual>
-    <collision>
-      <geometry>
-        <mesh filename="package://experiment_settings/meshes/collision/shoulder.stl"/>
-      </geometry>
-    </collision>
-    <inertial>
-      <mass value="3.7"/>
-      <origin rpy="0 0 0" xyz="0.0 0.0 0.0"/>
-      <inertia ixx="0.010267495893" ixy="0.0" ixz="0.0" iyy="0.010267495893" iyz="0.0" izz="0.00666"/>
-    </inertial>
-  </link>
-  <joint name="shoulder_lift_joint" type="revolute">
-    <parent link="shoulder_link"/>
-    <child link="upper_arm_link"/>
-    <origin rpy="0.0 1.5707963267948966 0.0" xyz="0.0 0.138 0.0"/>
-    <axis xyz="0 1 0"/>
-    <limit effort="150.0" lower="-3.141592653589793" upper="3.141592653589793" velocity="3.14"/>
-    <dynamics damping="0.0" friction="0.0"/>
-  </joint>
-  <link name="upper_arm_link">
-    <visual>
-      <geometry>
-        <mesh filename="package://experiment_settings/meshes/visual/upperarm.dae"/>
-      </geometry>
-      <material name="LightGrey">
-        <color rgba="0.7 0.7 0.7 1.0"/>
-      </material>
-    </visual>
-    <collision>
-      <geometry>
-        <mesh filename="package://experiment_settings/meshes/collision/upperarm.stl"/>
-      </geometry>
-    </collision>
-    <inertial>
-      <mass value="8.393"/>
-      <origin rpy="0 0 0" xyz="0.0 0.0 0.2125"/>
-      <inertia ixx="0.1338857818623325" ixy="0.0" ixz="0.0" iyy="0.1338857818623325" iyz="0.0" izz="0.0151074"/>
-    </inertial>
-  </link>
-  <joint name="elbow_joint" type="revolute">
-    <parent link="upper_arm_link"/>
-    <child link="forearm_link"/>
-    <origin rpy="0.0 0.0 0.0" xyz="0.0 -0.131 0.425"/>
-    <axis xyz="0 1 0"/>
-    <limit effort="150.0" lower="-3.141592653589793" upper="3.141592653589793" velocity="3.14"/>
-    <dynamics damping="0.0" friction="0.0"/>
-  </joint>
-  <link name="forearm_link">
-    <visual>
-      <geometry>
-        <mesh filename="package://experiment_settings/meshes/visual/forearm.dae"/>
-      </geometry>
-      <material name="LightGrey">
-        <color rgba="0.7 0.7 0.7 1.0"/>
-      </material>
-    </visual>
-    <collision>
-      <geometry>
-        <mesh filename="package://experiment_settings/meshes/collision/forearm.stl"/>
-      </geometry>
-    </collision>
-    <inertial>
-      <mass value="2.275"/>
-      <origin rpy="0 0 0" xyz="0.0 0.0 0.196"/>
-      <inertia ixx="0.031179620861480004" ixy="0.0" ixz="0.0" iyy="0.031179620861480004" iyz="0.0" izz="0.004095"/>
-    </inertial>
-  </link>
-  <joint name="wrist_1_joint" type="revolute">
-    <parent link="forearm_link"/>
-    <child link="wrist_1_link"/>
-    <origin rpy="0.0 1.5707963267948966 0.0" xyz="0.0 0.0 0.392"/>
-    <axis xyz="0 1 0"/>
-    <limit effort="28.0" lower="-3.141592653589793" upper="3.141592653589793" velocity="6.28"/>
-    <dynamics damping="0.0" friction="0.0"/>
-  </joint>
-  <link name="wrist_1_link">
-    <visual>
-      <geometry>
-        <mesh filename="package://experiment_settings/meshes/visual/wrist1.dae"/>
-      </geometry>
-      <material name="LightGrey">
-        <color rgba="0.7 0.7 0.7 1.0"/>
-      </material>
-    </visual>
-    <collision>
-      <geometry>
-        <mesh filename="package://experiment_settings/meshes/collision/wrist1.stl"/>
-      </geometry>
-    </collision>
-    <inertial>
-      <mass value="1.219"/>
-      <origin rpy="0 0 0" xyz="0.0 0.127 0.0"/>
-      <inertia ixx="0.0025598989760400002" ixy="0.0" ixz="0.0" iyy="0.0025598989760400002" iyz="0.0" izz="0.0021942"/>
-    </inertial>
-  </link>
-  <joint name="wrist_2_joint" type="revolute">
-    <parent link="wrist_1_link"/>
-    <child link="wrist_2_link"/>
-    <origin rpy="0.0 0.0 0.0" xyz="0.0 0.127 0.0"/>
-    <axis xyz="0 0 1"/>
-    <limit effort="28.0" lower="-3.141592653589793" upper="3.141592653589793" velocity="6.28"/>
-    <dynamics damping="0.0" friction="0.0"/>
-  </joint>
-  <link name="wrist_2_link">
-    <visual>
-      <geometry>
-        <mesh filename="package://experiment_settings/meshes/visual/wrist2.dae"/>
-      </geometry>
-      <material name="LightGrey">
-        <color rgba="0.7 0.7 0.7 1.0"/>
-      </material>
-    </visual>
-    <collision>
-      <geometry>
-        <mesh filename="package://experiment_settings/meshes/collision/wrist2.stl"/>
-      </geometry>
-    </collision>
-    <inertial>
-      <mass value="1.219"/>
-      <origin rpy="0 0 0" xyz="0.0 0.0 0.1"/>
-      <inertia ixx="0.0025598989760400002" ixy="0.0" ixz="0.0" iyy="0.0025598989760400002" iyz="0.0" izz="0.0021942"/>
-    </inertial>
-  </link>
-  <joint name="wrist_3_joint" type="revolute">
-    <parent link="wrist_2_link"/>
-    <child link="wrist_3_link"/>
-    <origin rpy="0.0 0.0 0.0" xyz="0.0 0.0 0.1"/>
-    <axis xyz="0 1 0"/>
-    <limit effort="28.0" lower="-3.141592653589793" upper="3.141592653589793" velocity="6.28"/>
-    <dynamics damping="0.0" friction="0.0"/>
-  </joint>
-  <link name="wrist_3_link">
-    <visual>
-      <geometry>
-        <mesh filename="package://experiment_settings/meshes/visual/wrist3.dae"/>
-      </geometry>
-      <material name="LightGrey">
-        <color rgba="0.7 0.7 0.7 1.0"/>
-      </material>
-    </visual>
-    <collision>
-      <geometry>
-        <mesh filename="package://experiment_settings/meshes/collision/wrist3.stl"/>
-      </geometry>
-    </collision>
-    <inertial>
-      <mass value="0.1879"/>
-      <origin rpy="1.5707963267948966 0 0" xyz="0.0 0.0771 0.0"/>
-      <inertia ixx="9.890410052167731e-05" ixy="0.0" ixz="0.0" iyy="9.890410052167731e-05" iyz="0.0" izz="0.0001321171875"/>
-    </inertial>
-  </link>
-  <joint name="ee_fixed_joint" type="fixed">
-    <parent link="wrist_3_link"/>
+  <xacro:include filename="$(find ur_description)/urdf/inc/ur_macro.xacro"/>
+  <xacro:ur_robot
+    prefix=""
+    joint_limits_parameters_file="$(find ur_description)/config/ur5e/joint_limits.yaml"
+    kinematics_parameters_file="$(find ur_description)/config/ur5e/default_kinematics.yaml"
+    physical_parameters_file="$(find ur_description)/config/ur5e/physical_parameters.yaml"
+    visual_parameters_file="$(find ur_description)/config/ur5e/visual_parameters.yaml"
+    transmission_hw_interface="hardware_interface/EffortJointInterface"
+    safety_limits="false"
+    safety_pos_margin="0.15"
+    safety_k_position="20"
+  />
+  <link name="ee_link"/>
+  <joint name="tool0_ee_link" type="fixed">
+    <parent link="tool0"/>
     <child link="ee_link"/>
-    <origin rpy="0.0 0.0 1.5707963267948966" xyz="0.0 0.1 0.0"/>
-  </joint>
-  <link name="ee_link">
-    <collision>
-      <geometry>
-        <box size="0.01 0.01 0.01"/>
-      </geometry>
-      <origin rpy="0 0 0" xyz="-0.01 0 0"/>
-    </collision>
-    <inertial>
-      <mass value="0.1" />
-      <origin xyz="0 0 0" rpy="0 0 0" />
-      <inertia ixx="0.03" iyy="0.03" izz="0.03" ixy="0.0" ixz="0.0" iyz="0.0" />
-    </inertial>
-  </link>
-  <transmission name="shoulder_pan_trans">
-    <type>transmission_interface/SimpleTransmission</type>
-    <joint name="shoulder_pan_joint">
-      <hardwareInterface>hardware_interface/EffortJointInterface</hardwareInterface>
-    </joint>
-    <actuator name="shoulder_pan_motor">
-      <mechanicalReduction>1</mechanicalReduction>
-      <hardwareInterface>hardware_interface/EffortJointInterface</hardwareInterface>
-    </actuator>
-  </transmission>
-  <transmission name="shoulder_lift_trans">
-    <type>transmission_interface/SimpleTransmission</type>
-    <joint name="shoulder_lift_joint">
-      <hardwareInterface>hardware_interface/EffortJointInterface</hardwareInterface>
-    </joint>
-    <actuator name="shoulder_lift_motor">
-      <mechanicalReduction>1</mechanicalReduction>
-      <hardwareInterface>hardware_interface/EffortJointInterface</hardwareInterface>
-    </actuator>
-  </transmission>
-  <transmission name="elbow_trans">
-    <type>transmission_interface/SimpleTransmission</type>
-    <joint name="elbow_joint">
-      <hardwareInterface>hardware_interface/EffortJointInterface</hardwareInterface>
-    </joint>
-    <actuator name="elbow_motor">
-      <mechanicalReduction>1</mechanicalReduction>
-      <hardwareInterface>hardware_interface/EffortJointInterface</hardwareInterface>
-    </actuator>
-  </transmission>
-  <transmission name="wrist_1_trans">
-    <type>transmission_interface/SimpleTransmission</type>
-    <joint name="wrist_1_joint">
-      <hardwareInterface>hardware_interface/EffortJointInterface</hardwareInterface>
-    </joint>
-    <actuator name="wrist_1_motor">
-      <mechanicalReduction>1</mechanicalReduction>
-      <hardwareInterface>hardware_interface/EffortJointInterface</hardwareInterface>
-    </actuator>
-  </transmission>
-  <transmission name="wrist_2_trans">
-    <type>transmission_interface/SimpleTransmission</type>
-    <joint name="wrist_2_joint">
-      <hardwareInterface>hardware_interface/EffortJointInterface</hardwareInterface>
-    </joint>
-    <actuator name="wrist_2_motor">
-      <mechanicalReduction>1</mechanicalReduction>
-      <hardwareInterface>hardware_interface/EffortJointInterface</hardwareInterface>
-    </actuator>
-  </transmission>
-  <transmission name="wrist_3_trans">
-    <type>transmission_interface/SimpleTransmission</type>
-    <joint name="wrist_3_joint">
-      <hardwareInterface>hardware_interface/EffortJointInterface</hardwareInterface>
-    </joint>
-    <actuator name="wrist_3_motor">
-      <mechanicalReduction>1</mechanicalReduction>
-       <hardwareInterface>hardware_interface/EffortJointInterface</hardwareInterface>
-    </actuator>
-  </transmission>
+    <origin xyz="0 0 0" rpy="0 0 0"/>
+  </joint>
   <gazebo reference="shoulder_link">
     <selfCollide>true</selfCollide>
@@ -327,37 +79,8 @@
     <selfCollide>true</selfCollide>
   </gazebo>
-  <!-- ROS base_link to UR 'Base' Coordinates transform -->
-  <link name="base"/>
-  <joint name="base_link-base_fixed_joint" type="fixed">
-    <!-- NOTE: this rotation is only needed as long as base_link itself is
-                 not corrected wrt the real robot (ie: rotated over 180
-                 degrees)
-      -->
-    <origin rpy="0 0 -3.141592653589793" xyz="0 0 0"/>
-    <parent link="base_link"/>
-    <child link="base"/>
-  </joint>
-  <!-- Frame coincident with all-zeros TCP on UR controller -->
-  <link name="tool0"/>
-  <joint name="wrist_3_link-tool0_fixed_joint" type="fixed">
-    <origin rpy="-1.5707963267948966 0 0" xyz="0 0.1 0"/>
-    <parent link="wrist_3_link"/>
-    <child link="tool0"/>
-  </joint>
   <material name="camera_aluminum">
     <color rgba="0.5 0.5 0.5 1"/>
   </material>
   <!-- camera body, with origin at bottom screw mount -->
-  <joint name="camera_joint" type="fixed">
-    <origin rpy="3.1414 0.0 1.5707" xyz="0.05472 0.014 0.03"/>
-    <parent link="ur_gripper"/>
-    <child link="camera_bottom_screw_frame"/>
-  </joint>
-  <link name="camera_bottom_screw_frame"/>
-  <joint name="camera_link_joint" type="fixed">
-    <origin rpy="0 0 0" xyz="0 0.0175 0.0125"/>
-    <parent link="camera_bottom_screw_frame"/>
-    <child link="camera_link"/>
-  </joint>
   <link name="camera_link">
     <visual>
@@ -1120,15 +843,30 @@
     <parent link="base_cylinder"/>
     <child link="base_link"/>
-    <origin rpy="0.0 0.0 0.0" xyz="0.0 0.0 0.35"/>
+    <origin rpy="0.0 0.0 -1.57" xyz="0.0 0.0 0.35"/>
+  </joint>
+  <joint name="camera_joint" type="fixed">
+    <origin rpy="3.1414 0.0 1.5707" xyz="0.055 0.015 0.03"/>
+    <!-- <origin rpy="0.0 -0.0 0.0" xyz="-0.0 -0.0 -0.0"/> -->
+    <parent link="ur_gripper"/>
+    <child link="camera_bottom_screw_frame"/>
+  </joint>
+  <link name="camera_bottom_screw_frame"/>
+  <joint name="camera_link_joint" type="fixed">
+    <origin rpy="0 0 0" xyz="0 0.0175 0.0125"/>
+    <!-- <origin rpy="0.0 -0.0 0.0" xyz="-0.0 -0.0 -0.0"/> -->
+    <parent link="camera_bottom_screw_frame"/>
+    <child link="camera_link"/>
   </joint>
   <joint name="ur_gripper_joint" type="fixed">
-    <parent link="ee_link"/>
+    <parent link="wrist_3_link"/>
     <child link="ur_gripper"/>
-    <origin rpy="0.0 -0.7854 -1.57" xyz="-0.002 -0.08423 -0.15968"/>
+    <!-- <origin rpy="1.57 -0.7854 -1.57" xyz="-0.002 -0.08423 -0.15968"/> -->
+    <origin rpy="1.57 -0.0 -0.785" xyz="0.08423 0.161 -0.0"/><!-- 0.055 0.175 -->
   </joint>
   <joint name="urGripper_gripper_joint" type="fixed">
     <parent link="ur_gripper"/>
     <child link="robotiq_palm"/>
-    <origin rpy="0.0 3.1415 0.0" xyz="0.05355 0.05 0.17247"/>
+    <!-- <origin rpy="0.0 3.1415 0.0" xyz="0.05355 0.05 0.17247"/> -->
+    <origin rpy="0.0 3.14 0.0" xyz="0.055 0.068 0.1735"/>
   </joint>
   <joint name="world_table_joint" type="fixed">

Commit message: Update ur5e_sim.xacro

File: catkin_ws/src/experiment_settings/urdf/ur5e_sim.xacro (robot description, xacro)
@@ -40,4 +40,11 @@
   <!--property name="wrist_3_length" value="0.0823" /-->
   <!-- manually measured -->
+  <!-- <link name="root"/>
+  <joint name="root2world" type="fixed">
+    <parent link="root"/>
+    <child link="world"/>
+    <origin xyz="0 0 0" rpy="0 0 0"/>
+  </joint>
+   -->
   <xacro:include filename="$(find ur_description)/urdf/inc/ur_macro.xacro"/>
   <xacro:ur_robot
